Commit message: removed hands

File: urdf/human.urdf.xacro (robot description, xacro)
@@ -2,17 +2,3 @@
 <robot name="human" xmlns:xacro="http://www.ros.org/wiki/xacro">
     <link name="robot_root"></link>
-    <joint name="hand_1_joint" type="floating">
-      <parent link="robot_root"/>
-      <child link="hand_1"/>
-      <origin xyz="0.0 0.0 0.0" rpy="0   0   0"/>
-    </joint>
-   <link name="hand_1">
-    </link>
-    <joint name="hand_2_joint" type="floating">
-      <parent link="robot_root"/>
-      <child link="hand_2"/>
-      <origin xyz="0.0 0.0 0.0" rpy="0   0   0"/>
-    </joint>
-   <link name="hand_2">
-    </link>
 </robot>
